File: main-board.sch (EAGLE design)
At the start: 1 part

Commit message: create power managment
Parts:
- added C1, C2, C4: 10uF, SparkFun-Capacitors:10UF-0805-10V-10%
- added C3: 1.0uF, SparkFun-Capacitors:1.0UF-0805-25V-(+80/-20%)
- added D1: Yellow, SparkFun-LED:LED-YELLOW0603
- added D2: (no value), adafruit:DIODESOD-123
- added J1: (no value), SparkFun-Connectors:JST_2MM_MALE
- added R1: 4.7k, SparkFun-Resistors:4.7KOHM-0603-1/10W-1%
- added R2: 1k, SparkFun-Resistors:1KOHM-0603-1/10W-1%
- added R3, R4: 100k, SparkFun-Resistors:100KOHM-0603-1/10W-1%
- added U2: ESP32-WROOM-32D, SnapEDA-Library:ESP32-WROOM-32D
- added U3: CP2104-F03-GM, SnapEDA-Library:CP2104-F03-GM
- added U4: AP2112K-3.3TRG1, SnapEDA-Library:AP2112K-3.3TRG1
- added U5: MCP73831-2ACI/MC, SnapEDA-Library:MCP73831-2ACI/MC
- added U6: DMG3415U-7, SnapEDA-Library:DMG3415U-7
- U1: OC_NEWARK (none) -> unknown
Connections:
- new net 3.3V: C2.1, C3.1, U4.VOUT
- new net GND: C1.2, C2.2, C3.2, C4.2, J1.-, R1.2, R3.1, U2.GND, U3.GND, U4.GND, U5.VSS
- new net N$1: R1.1, U5.PROG
- new net N$2: R2.2, U5.STAT
- new net N$3: D1.C, R2.1
- new net N$4: C4.1, D2.C, R4.1, U4.VIN, U6.D
- new net N$5: R4.2, U4.EN
- new net USBRX: U2.RXD0, U3.TXD
- new net USBTX: U2.TXD0, U3.RXD
- new net VCC: D1.A, D2.A, R3.2, U5.VDD, U6.G
- new net V_BATT: C1.1, J1.+, U5.VBAT, U6.S
Other:
- moved on the sheet: U1

Commit message: added board
Parts:
- added BT1: (no value), SparkFun-Batteries:BATTERY-20MM_PTH
- added C5: 0.1uF, SparkFun-Capacitors:0.1UF-0603-25V-(+80/-20%)
- added C6: 10uF, SparkFun-Capacitors:10UF-0805-10V-10%
- added D3: BLUE, SparkFun-LED:LED-BLUE0603
- added J2: (no value), SparkFun-Connectors:USB_MICRO-B_FEMALE-SMT
- added R5: 1k, SparkFun-Resistors:1KOHM-0603-1/10W-1%
- added U7: DMG3415U-7, SnapEDA-Library:DMG3415U-7
Connections:
- new net GPSENABLE: U2.IO17, U7.G
- new net GPSRX: U1.TX, U2.IO19
- new net GPSTX: U1.RX, U2.IO18
- new net N$10: J2.D-, U3.D-
- new net N$6: C5.1, U1.VCC, U7.D
- new net N$7: D3.A, U1.3D-FIX
- new net N$8: D3.C, R5.2
- new net N$9: J2.D+, U3.D+
- new net REGIN: C6.1, U3.REGIN, U3.VDD, U3.VIO
- new net VBACKUP: BT1.+, U1.VBACKUP
- net 3.3V: now also U7.S
- net GND: now also BT1.-, C5.2, C6.2, J2.GND, R5.1, U1.GND@1, U1.GND@2, U1.GND@3, U1.GND@4
- net VCC: now also J2.VBUS, U3.VBUS
Other:
- moved on the sheet: U1, U2, U3

Commit message: added board design
Connections:
- net 3.3V: now also U2.3V3
Other:
- moved on the sheet: U2
Changed lines of the file:
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@@
 <part name="C6" library="SparkFun-Capacitors" library_urn="urn:adsk.eagle:library:510" deviceset="10UF" device="-0805-10V-10%" package3d_urn="urn:adsk.eagle:package:37429/1" value="10uF"/>
 <part name="GND12" library="supply1" library_urn="urn:adsk.eagle:library:371" deviceset="GND" device=""/>
+<part name="SUPPLY11" library="SparkFun-PowerSymbols" library_urn="urn:adsk.eagle:library:530" deviceset="3.3V" device=""/>
 </parts>
 <sheets>
@@
 <attribute name="MPN" x="137.16" y="17.78" size="1.778" layer="96" display="off"/>
 </instance>
-<instance part="U2" gate="G$1" x="-55.88" y="-7.62" smashed="yes">
-<attribute name="NAME" x="-70.9159" y="29.0545" size="1.783840625" layer="95"/>
-<attribute name="VALUE" x="-71.1667" y="-45.8281" size="1.78345" layer="96"/>
+<instance part="U2" gate="G$1" x="299.72" y="71.12" smashed="yes">
+<attribute name="NAME" x="284.6841" y="107.7945" size="1.783840625" layer="95"/>
+<attribute name="VALUE" x="284.4333" y="32.9119" size="1.78345" layer="96"/>
 </instance>
 <instance part="U3" gate="G$1" x="213.36" y="109.22" smashed="yes">
@@
 <attribute name="VALUE" x="101.6" y="83.82" size="1.778" layer="96"/>
 </instance>
-<instance part="GND3" gate="1" x="-33.02" y="-45.72" smashed="yes">
-<attribute name="VALUE" x="-35.56" y="-48.26" size="1.778" layer="96"/>
+<instance part="GND3" gate="1" x="322.58" y="33.02" smashed="yes">
+<attribute name="VALUE" x="320.04" y="30.48" size="1.778" layer="96"/>
 </instance>
 <instance part="GND4" gate="1" x="119.38" y="127" smashed="yes">
@@
 <instance part="GND12" gate="1" x="185.42" y="96.52" smashed="yes">
 <attribute name="VALUE" x="182.88" y="93.98" size="1.778" layer="96"/>
+</instance>
+<instance part="SUPPLY11" gate="G$1" x="325.12" y="104.14" smashed="yes" rot="R270">
+<attribute name="VALUE" x="327.914" y="104.14" size="1.778" layer="96" rot="R270" align="bottom-center"/>
 </instance>
 </instances>
@@
 <segment>
 <pinref part="U2" gate="G$1" pin="TXD0"/>
-<wire x1="-73.66" y1="2.54" x2="-81.28" y2="2.54" width="0.1524" layer="91"/>
-<label x="-83.82" y="2.54" size="1.778" layer="95"/>
+<wire x1="281.94" y1="81.28" x2="274.32" y2="81.28" width="0.1524" layer="91"/>
+<label x="271.78" y="81.28" size="1.778" layer="95"/>
 </segment>
 <segment>
@@
 <segment>
 <pinref part="U2" gate="G$1" pin="RXD0"/>
-<wire x1="-73.66" y1="0" x2="-81.28" y2="0" width="0.1524" layer="91"/>
-<label x="-83.82" y="0" size="1.778" layer="95"/>
+<wire x1="281.94" y1="78.74" x2="274.32" y2="78.74" width="0.1524" layer="91"/>
+<label x="271.78" y="78.74" size="1.778" layer="95"/>
 </segment>
 <segment>
@@
 <pinref part="U2" gate="G$1" pin="GND"/>
 <pinref part="GND3" gate="1" pin="GND"/>
-<wire x1="-38.1" y1="-40.64" x2="-33.02" y2="-40.64" width="0.1524" layer="91"/>
-<wire x1="-33.02" y1="-40.64" x2="-33.02" y2="-43.18" width="0.1524" layer="91"/>
+<wire x1="317.5" y1="38.1" x2="322.58" y2="38.1" width="0.1524" layer="91"/>
+<wire x1="322.58" y1="38.1" x2="322.58" y2="35.56" width="0.1524" layer="91"/>
 </segment>
 <segment>
@@
 <wire x1="58.42" y1="45.72" x2="66.04" y2="45.72" width="0.1524" layer="91"/>
 </segment>
+<segment>
+<pinref part="U2" gate="G$1" pin="3V3"/>
+<pinref part="SUPPLY11" gate="G$1" pin="3.3V"/>
+<wire x1="317.5" y1="104.14" x2="325.12" y2="104.14" width="0.1524" layer="91"/>
+</segment>
 </net>
 <net name="N$4" class="0">
@@
 <segment>
 <pinref part="U2" gate="G$1" pin="IO18"/>
-<wire x1="-38.1" y1="-5.08" x2="-30.48" y2="-5.08" width="0.1524" layer="91"/>
-<label x="-33.02" y="-5.08" size="1.778" layer="95"/>
+<wire x1="317.5" y1="73.66" x2="325.12" y2="73.66" width="0.1524" layer="91"/>
+<label x="322.58" y="73.66" size="1.778" layer="95"/>
 </segment>
 <segment>
@@
 <segment>
 <pinref part="U2" gate="G$1" pin="IO19"/>
-<wire x1="-38.1" y1="-7.62" x2="-30.48" y2="-7.62" width="0.1524" layer="91"/>
-<label x="-33.02" y="-7.62" size="1.778" layer="95"/>
+<wire x1="317.5" y1="71.12" x2="325.12" y2="71.12" width="0.1524" layer="91"/>
+<label x="322.58" y="71.12" size="1.778" layer="95"/>
 </segment>
 <segment>
@@
 <segment>
 <pinref part="U2" gate="G$1" pin="IO17"/>
-<wire x1="-38.1" y1="-2.54" x2="-30.48" y2="-2.54" width="0.1524" layer="91"/>
-<label x="-33.02" y="-2.54" size="1.778" layer="95"/>
-</segment>
-<segment>
+<wire x1="317.5" y1="76.2" x2="325.12" y2="76.2" width="0.1524" layer="91"/>
+<label x="322.58" y="76.2" size="1.778" layer="95"/>
+</segment>
+<segment>
