File: main-board.brd (EAGLE design)
At the start: 100 x 80 mm, 24 parts, among them U2 ESP32-WROOM-32D, U3 CP2104-F03-GM, U4 AP2112K-3.3TRG1, U5 MCP73831-2ACI/MC, U6 DMG3415U-7, U7 DMG3415U-7

Commit message: added board
Parts:
- removed D3: BLUE, SparkFun-LED:LED-0603
- removed R5: 1k, SparkFun-Resistors:0603
- removed U1: (no value), adafruit:FGPMMOPA6H
- added IC1: SAM-M8Q, hermes-parts:SAM-M8Q
- moved U4 59.7 mm to (22.9, 47.0)
- moved D2 53.6 mm to (14.0, 48.3)
- moved U2 47.6 mm to (22.9, 64.8)
- moved U3 36.9 mm to (40.6, 63.5), turned to 270 degrees
- moved U6 24.1 mm to (31.8, 43.2)
- moved J1 22.9 mm to (40.6, 34.3)
- moved U5 18.2 mm to (39.4, 20.3)
- moved D1 14.5 mm to (85.1, 41.9)
- moved U7 14.2 mm to (31.8, 22.9)
- moved R4 12.5 mm to (88.9, 41.9)
- moved R2 12.5 mm to (96.5, 41.9)
- moved R3 12.5 mm to (92.7, 41.9)
- moved C5 12.5 mm to (53.3, 34.3)
- moved C1 12.5 mm to (72.4, 34.3)
- moved C2 12.5 mm to (68.6, 34.3)
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Connections:
- removed net N$8: D3.C, R5.2
- removed net VBACKUP: BT1.1, U1.P$4
- net GND: now also IC1.1, IC1.10, IC1.11, IC1.15, IC1.16, IC1.20, IC1.4, IC1.5, IC1.6; no longer R5.1, U1.P$12, U1.P$19, U1.P$3, U1.P$8
- net GPSRX: now also IC1.13; no longer U1.P$9
- net GPSTX: now also IC1.14; no longer U1.P$10
- net N$6: now also IC1.17, IC1.2; no longer U1.P$1
- net N$7: now also BT1.1, IC1.3; no longer D3.A, U1.P$5
Routing:
- net GND: track 311.7 -> 0.00 mm, vias 3 -> 0
- net VCC: track 115.4 -> 0.00 mm, vias 3 -> 0
- net N$4: track 85.8 -> 0.00 mm, vias 4 -> 0
- net GPSTX: track 85.5 -> 0.00 mm
- net N$7: track 81.5 -> 0.00 mm
- net V_BATT: track 68.2 -> 0.00 mm, vias 2 -> 0
- net N$6: track 64.7 -> 0.00 mm, vias 3 -> 0
- net 3.3V: track 61.3 -> 0.00 mm
- net GPSRX: track 57.0 -> 0.00 mm, vias 2 -> 0
- net N$2: track 51.9 -> 0.00 mm
- net N$9: track 44.3 -> 0.00 mm, vias 2 -> 0
- net REGIN: track 40.6 -> 0.00 mm
- net GPSENABLE: track 36.5 -> 0.00 mm
- net N$1: track 34.7 -> 0.00 mm
- net VBACKUP: track 33.5 -> 0.00 mm
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Other:
- board size 100 x 80 mm -> 45.4 x 80 mm
