File: hermes-control.brd (EAGLE design)
At the start: 110 x 50 mm, 52 parts, among them Q1 600mA/40V, U1 LSM9DS1TR, U2 ESP32-WROOM-32D, U3 CP2104-F03-GM, U4 AP2112K-3.3TRG1, U5 MCP73831-2ACI/MC, U6 DMG3415U-7, U7 DMG3415U-7

Commit message: updated componets to match bom
Parts:
- removed D2: (no value), adafruit:SOD-123
- removed D3, D4, D5, D6: BLUE, SparkFun-LED:LED-1206
- removed J1: (no value), SparkFun-Connectors:JST-2-SMD
- removed U$2: MICROSD, adafruit:MICROSD
- added BLUE1, BLUE2, BLUE3, BLUE4: LTST-C190TBKT, hermes:0603
- added J3: 2201778-1, hermes:TE_2201778-1
- added LBAT: S2B-PH-SM4-TB(LF)(SN), hermes:JST_S2B-PH-SM4-TB(LF)(SN)
- BT1: value (none) -> BK-5067; device SparkFun-Batteries:BATTCON_12MM -> hermes:BAT_BK-5067
- C1, C2, C4, C6, C7: value 10uF -> EMK107BBJ106MA-T; device SparkFun-Capacitors:0805 -> hermes:EMK107BBJ106MA-T_CAPC1608X95N
- C3: value 1.0uF -> GMK107AB7105KAHT; device SparkFun-Capacitors:0805 -> hermes:CAPC1608X90N
- C5, C8: value 0.1uF -> CL21B104KBCNNNC; device SparkFun-Capacitors:0603 -> hermes:CAPC2012X140N
- C9: value 4.7uF -> JMK107BJ475KA-T; device SparkFun-Capacitors:0603 -> hermes:CAPC1608X95N
- D1: device SparkFun-LED:LED-0603 -> hermes:LEDSC160X80X70L45N
- Q1: value 600mA/40V -> MMBT2222A; device SparkFun-DiscreteSemi:SOT23-3 -> hermes:SOT23
- R1, R15, R16, R5, R6: value 4.7k -> ERJ-XGNF4701Y; device SparkFun-Resistors:0603 -> hermes:RESC1005X40
- R10, R11, R12, R13, R14, R9: value 10k -> RP73PF1J10KBTDF; device SparkFun-Resistors:0603 -> hermes:RESC1608X50N
- R2: value 1k -> CPF0402B1K0E1; device SparkFun-Resistors:0603 -> hermes:CPF0402B1K0E1_RESC1005X35N
- R3, R4: value 100k -> CPF0402B100KE1; device SparkFun-Resistors:0603 -> hermes:RESC1005X35N
- R7, R8: value 100K -> CPF0402B100KE1; device SparkFun-Resistors:0402 -> hermes:RESC1005X35N
- S1, S2: value MOMENTARY-SWITCH-SPST-PTH-6.0MM -> 1825910-7; device SparkFun-Switches:TACTILE_SWITCH_PTH_6.0MM -> hermes:SW_1825910-7
- moved R16 390.9 mm to (-0.43, -307.3)
- moved R15 377.9 mm to (-0.43, -294.6)
- moved R7 366.4 mm to (-0.46, -281.9)
- moved R8 354.2 mm to (-0.46, -269.2)
- moved R9 337.5 mm to (-0.79, -256.5)
- moved R10 325.2 mm to (-0.79, -243.8)
- moved S2 321.9 mm to (-102.9, -251.5)
- moved BT1 306.4 mm to (-82.5, -231.1)
- moved C8 299.4 mm to (-0.90, -218.1)
- moved C9 287.7 mm to (-0.80, -205.4)
- moved C7 273.1 mm to (-0.80, -192.7)
- moved C5 261.3 mm to (-0.90, -180.0)
- moved Q1 241.3 mm to (-0.95, -166.2)
- moved R6 233.5 mm to (-0.43, -152.4)
- moved R5 220.5 mm to (-0.43, -139.7)
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Connections:
- removed net GND1: U$2.MT1, U$2.MT2
- net 3.3V: now also J3.4, S1.4; no longer S1.3, U$2.4
- net CS: now also J3.2; no longer U$2.2
- net DIN: now also J3.3; no longer U$2.3
- net DOUT: now also J3.7; no longer U$2.7
- net GND: now also BLUE1.1, BLUE2.1, BLUE3.1, BLUE4.1, BT1.NEG, J3.11, J3.12, J3.13, J3.14, J3.15, J3.16, J3.6, LBAT.1; no longer BT1.GND, D3.C, D4.C, D5.C, D6.C, J1.1
- net N$11: now also BLUE1.2; no longer D3.A
- net N$13: now also BLUE2.2; no longer D4.A
- net N$14: now also BLUE3.2; no longer D5.A
- net N$15: now also BLUE4.2; no longer D6.A
- net N$4: no longer D2.C
- net N$7: now also BT1.POS1, BT1.POS2; no longer BT1.PWR@1
- net SCLK: now also J3.5; no longer U$2.5
- net USER: now also S2.2; no longer S2.1
- net VCC: no longer D2.A
- net V_BATT: now also LBAT.2; no longer J1.2
Routing:
- net N$13: track 2.81 -> 0.96 mm
- net N$15: track 2.81 -> 0.96 mm
- net N$14: track 2.81 -> 0.96 mm
- net N$11: track 2.81 -> 0.96 mm

Commit message: started to wries a few things
Parts:
- added C10, C12, C14: CL21B104KBCNNNC, hermes:CAPC2012X140N
- added C11, C13: EMK107BBJ106MA-T, hermes:EMK107BBJ106MA-T_CAPC1608X95N
- added R17, R18, R19, R20: RP73PF1J10KBTDF, hermes:RESC1608X50N
- moved S2 323.1 mm to (17.8, 48.3)
- moved BT1 318.7 mm to (83.8, 40.6), flipped to the bottom, turned to 270 degrees
- moved C3 148.7 mm to (27.2, 31.8), turned to 90 degrees
- moved C2 135.7 mm to (24.6, 31.8), turned to 90 degrees
- moved R4 118.6 mm to (19.9, 27.9), turned to 270 degrees
- moved J3 118.1 mm to (36.8, 24.1), turned to 180 degrees
- moved C4 110.3 mm to (22.1, 31.8), turned to 270 degrees
- moved LBAT 105.6 mm to (11.4, 29.2), turned to 270 degrees
- moved R3 98.5 mm to (11.0, 34.3)
- moved C1 79.2 mm to (15.7, 26.7)
- moved J2 74.9 mm to (12.7, 17.8)
- moved U5 73.9 mm to (16.5, 29.2), turned to 0 degrees
- moved U6 73.8 mm to (15.2, 33.0)
- moved R1 72.1 mm to (17.4, 31.8), turned to 180 degrees
- moved U3 64.9 mm to (20.3, 22.9)
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Connections:
- removed net VDDIO: U1.1, U1.3
- new net N$10: R18.2, U1.8
- new net N$16: C14.1, U1.1, U1.3
- new net N$17: R19.1, U1.5
- new net N$18: R20.1, U1.6
- new net N$9: R17.2, U1.7
- net 3.3V: now also C12.1, C13.1, R17.1, R18.1, R19.2, R20.2, U3.8
- net GND: now also C12.2, C13.2, C14.2
- net SCL: now also U1.2
- net SDA: now also U1.4
- net VCC: no longer U3.8
Routing:
- net DIN: track 0.00 -> 61.4 mm, vias 0 -> 2
- net DOUT: track 0.00 -> 52.6 mm, vias 0 -> 2
- net CS: track 0.00 -> 51.4 mm, vias 0 -> 2
- net SCLK: track 0.00 -> 51.2 mm, vias 0 -> 2
- net TX1: track 0.00 -> 31.3 mm
- net VCC: track 0.00 -> 30.9 mm
- net RX1: track 0.00 -> 30.3 mm, vias 0 -> 2
- net 3.3V: track 0.00 -> 18.0 mm
- net N$4: track 0.00 -> 13.1 mm
- net V_BATT: track 0.00 -> 12.1 mm
- net D-: track 0.00 -> 9.78 mm, vias 0 -> 2
- net D+: track 0.00 -> 7.09 mm
- net N$2: track 0.00 -> 2.85 mm
- net N$5: track 0.00 -> 2.02 mm
- net N$1: track 0.00 -> 1.86 mm
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
Commit message: stuck trying to finish wiring
Parts:
- moved BLUE4 405.1 mm to (54.6, 45.7), turned to 180 degrees
- moved BLUE3 397.4 mm to (47.0, 45.7), turned to 180 degrees
- moved BLUE2 389.8 mm to (39.4, 45.7), turned to 180 degrees
- moved BLUE1 382.3 mm to (31.8, 45.7), turned to 180 degrees
- moved R16 354.2 mm to (83.4, 36.8)
- moved R15 344.4 mm to (83.4, 39.4)
- moved R7 307.7 mm to (13.5, 25.4), turned to 90 degrees
- moved R8 293.8 mm to (14.8, 24.1), turned to 270 degrees
- moved R9 292.2 mm to (80.5, 24.1), turned to 90 degrees
- moved R10 284.4 mm to (83.0, 27.9), turned to 90 degrees
- moved C8 281.7 mm to (51.2, 58.8), flipped to the bottom
- moved C9 271.7 mm to (51.3, 61.3), flipped to the bottom
- moved C7 232.7 mm to (25.9, 38.4), flipped to the bottom, turned to 270 degrees
- moved Q1 232.3 mm to (57.5, 58.6), flipped to the bottom, turned to 180 degrees
- moved R6 221.8 mm to (55.5, 62.2), flipped to the bottom
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Routing:
- net USBTX: track 0.00 -> 89.5 mm, vias 0 -> 4
- net USBRX: track 0.00 -> 84.5 mm
- net IO13: track 0.00 -> 67.5 mm, vias 0 -> 2
- net N$7: track 0.00 -> 62.0 mm
- net 3.3V: track 18.0 -> 58.7 mm, vias 0 -> 3
- net LED1: track 0.00 -> 28.1 mm
- net N$12: track 0.00 -> 20.8 mm
- net LED2: track 0.00 -> 20.3 mm
- net N$6: track 0.00 -> 16.7 mm
- net GND: track 0.00 -> 16.7 mm
- net DIN: track 61.4 -> 49.8 mm, vias 2 -> 1
- net LED3: track 1.05 -> 12.6 mm
- net DOUT: track 52.6 -> 43.1 mm, vias 2 -> 1
- net SCLK: track 51.2 -> 43.7 mm, vias 2 -> 1
- net USER: track 0.00 -> 5.73 mm, vias 0 -> 2
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
Commit message: everything is connected but ground
Parts:
- removed C10: CL21B104KBCNNNC, hermes:CAPC2012X140N
- removed C11: EMK107BBJ106MA-T, hermes:EMK107BBJ106MA-T_CAPC1608X95N
- moved C14 442.8 mm to (25.4, 55.2), turned to 180 degrees
- moved C13 440.6 mm to (27.6, 58.2), turned to 90 degrees
- moved C12 435.0 mm to (30.4, 58.0), turned to 90 degrees
- moved R20 411.6 mm to (32.1, 49.9), turned to 270 degrees
- moved R18 409.9 mm to (36.1, 49.9), turned to 90 degrees
- moved R19 409.5 mm to (29.8, 49.9), turned to 270 degrees
- moved R17 405.7 mm to (34.2, 49.9), turned to 90 degrees
- moved U1 21.4 mm to (33.3, 54.5)
- moved R10 7.82 mm to (77.3, 22.6)
- moved R16 6.48 mm to (83.4, 43.3)
- moved R9 4.95 mm to (75.5, 24.1)
- moved R5 3.05 mm to (58.0, 59.2)
- moved R6 3.05 mm to (55.5, 59.2)
- moved Q1 1.91 mm to (57.5, 56.7)
- moved R15 1.91 mm to (83.4, 41.3)
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Routing:
- net 3.3V: track 58.7 -> 299.4 mm, vias 3 -> 15
- net SCL: track 0.00 -> 179.2 mm, vias 0 -> 3
- net SDA: track 0.00 -> 163.6 mm, vias 0 -> 4
- net USER: track 5.73 -> 93.5 mm, vias 2 -> 6
- net CONFIG: track 3.68 -> 78.4 mm, vias 0 -> 4
- net GPSENABLE: track 0.00 -> 65.8 mm, vias 0 -> 3
- net GPSRX: track 0.00 -> 46.3 mm, vias 0 -> 1
- net GPSTX: track 0.00 -> 44.2 mm, vias 0 -> 1
- net LED1: track 28.1 -> 59.1 mm, vias 0 -> 2
- net TX2: track 0.73 -> 27.2 mm
- net N$7: track 62.0 -> 87.2 mm
- net LED2: track 20.3 -> 44.1 mm, vias 0 -> 2
- net LED4: track 4.79 -> 26.4 mm, vias 0 -> 2
- net RX2: track 0.22 -> 20.3 mm
- net LED3: track 12.6 -> 26.8 mm
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
Commit message: it is done
Parts:
- added C10: GMK107AB7105KAHT, hermes:CAPC1608X90N
- added Q2, Q3: MMBT2222A, hermes:SOT23
- added R21, R22, R23: RP73PF1J10KBTDF, hermes:RESC1608X50N
- added S3: 1825910-7, hermes:SW_1825910-7
- moved R4 0.85 mm to (19.1, 27.6)
Connections:
- new net DTR: Q2.2, R22.2, U3.23
- new net ESP_RST: C10.1, Q3.3, R23.1, S3.1, U2.3
- new net IO0: Q2.3, U2.25
- new net N$19: Q3.1, R22.1
- new net N$20: Q2.1, R21.1
- new net RTS: Q3.2, R21.2, U3.19
- net 3.3V: now also R23.2
- net CONFIG: now also U2.23; no longer U2.25
- net GND: now also C10.2, S3.4
Routing:
- net GND: track 16.7 -> 404.0 mm, vias 0 -> 40
- net RTS: track 0.00 -> 87.9 mm, vias 0 -> 4
- net ESP_RST: track 0.00 -> 86.3 mm, vias 0 -> 3
- net DTR: track 0.00 -> 81.0 mm, vias 0 -> 4
- net 3.3V: track 299.4 -> 322.2 mm
- net IO0: track 0.00 -> 11.6 mm, vias 0 -> 2
- net N$19: track 0.00 -> 7.75 mm, vias 0 -> 2
- net N$20: track 0.00 -> 6.66 mm, vias 0 -> 2
- net SCLK: track 37.6 -> 41.0 mm
- net N$4: track 13.1 -> 14.7 mm
- net LED1: track 59.1 -> 57.6 mm
- net CONFIG: track 78.4 -> 77.0 mm
- net N$5: track 2.02 -> 2.62 mm
- net N$2: track 2.85 -> 3.42 mm
- added copper zone on layer 1, net GND
- added copper zone on layer 16, net GND

Commit message: lets clean this up
Parts:
- added R24: 1k, rcl:R0603
- R2: value CPF0402B1K0E1 -> 1k; device hermes:CPF0402B1K0E1_RESC1005X35N -> rcl:R0603
Changed lines of the file:
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@@
 <drawing>
 <settings>
-<setting alwaysvectorfont="yes"/>
+<setting alwaysvectorfont="no"/>
 <setting verticaltext="up"/>
 </settings>
@@
 <attribute name="NAME" x="83.39" y="44.069" size="0.6096" layer="25" font="vector" ratio="20" align="bottom-center"/>
 </element>
-<element name="R2" library="hermes" package="CPF0402B1K0E1_RESC1005X35N" value="CPF0402B1K0E1" x="19.865" y="30.48" smashed="yes" rot="R180">
+<element name="R2" library="rcl" library_urn="urn:adsk.eagle:library:334" package="R0603" package3d_urn="urn:adsk.eagle:package:23555/3" value="1k" x="19.865" y="30.48" smashed="yes" rot="R180">
 <attribute name="NAME" x="19.865" y="29.718" size="0.6096" layer="25" font="vector" ratio="20" rot="R180" align="bottom-center"/>
+<attribute name="SPICEPREFIX" value="R" x="19.865" y="30.48" size="1.778" layer="27" rot="R180" display="off"/>
 </element>
 <element name="R3" library="hermes" package="RESC1005X35N" value="CPF0402B100KE1" x="10.975" y="34.29" smashed="yes">
@@
 <attribute name="NAME" x="49.73523125" y="21.109171875" size="0.528809375" layer="25" rot="R180"/>
 <attribute name="VALUE" x="49.728840625" y="23.630759375" size="0.526865625" layer="27" rot="R180"/>
+</element>
+<element name="R24" library="rcl" library_urn="urn:adsk.eagle:library:334" package="R0603" package3d_urn="urn:adsk.eagle:package:23555/3" value="1k" x="-10.668" y="8.763" smashed="yes">
+<attribute name="NAME" x="-11.303" y="9.398" size="1.27" layer="25"/>
+<attribute name="SPICEPREFIX" value="R" x="-10.668" y="8.763" size="1.778" layer="27" display="off"/>
+<attribute name="VALUE" x="-11.303" y="6.858" size="1.27" layer="27"/>
 </element>
 </elements>
@@
 <contactref element="U5" pad="5"/>
 <contactref element="R2" pad="2"/>
-<wire x1="19.41" y1="30.48" x2="19.836378125" y2="30.053621875" width="0.1524" layer="1"/>
+<wire x1="19.015" y1="30.48" x2="19.836378125" y2="30.053621875" width="0.1524" layer="1"/>
 <wire x1="19.836378125" y1="30.053621875" x2="19.836378125" y2="29.59760625" width="0.1524" layer="1"/>
 <wire x1="19.836378125" y1="29.59760625" x2="18.698771875" y2="28.46" width="0.1524" layer="1"/>
@@
 <contactref element="R2" pad="1"/>
 <contactref element="D1" pad="C"/>
-<wire x1="20.32" y1="30.48" x2="20.32" y2="31.75" width="0.1524" layer="1"/>
+<wire x1="20.715" y1="30.48" x2="20.32" y2="31.75" width="0.1524" layer="1"/>
 </signal>
 <signal name="N$4">

Commit message: replaced all componets with generics
Parts:
- removed BLUE1, BLUE2, BLUE3, BLUE4: LTST-C190TBKT, hermes:0603
- removed C9: JMK107BJ475KA-T, hermes:CAPC1608X95N
- removed D1: Yellow, hermes:LEDSC160X80X70L45N
- removed R12, R13, R14: RP73PF1J10KBTDF, hermes:RESC1608X50N
- removed R16, R6: ERJ-XGNF4701Y, hermes:RESC1005X40
- removed U6, U7: DMG3415U-7, SnapEDA-Library:SOT95P240X105-3N
- added C11: 10uF, rcl:C0603
- added LED1: Yellow, led:CHIPLED_0805
- added LED2, LED3, LED5: Blue, led:CHIPLED_0805
- added LED4: BLue, led:CHIPLED_0805
- added Q4: FDN360P, transistor-power:SUPER-SOT3
- added Q5: BC849SMD, transistor-npn:SOT23-BEC
- C1, C4, C6: value EMK107BBJ106MA-T -> 10uF; device hermes:EMK107BBJ106MA-T_CAPC1608X95N -> rcl:C0603
- C10: value GMK107AB7105KAHT -> 10uF; device hermes:CAPC1608X90N -> rcl:C0603
- C12, C5: value CL21B104KBCNNNC -> 0.1uF; device hermes:CAPC2012X140N -> rcl:C0603
- C13, C7: value EMK107BBJ106MA-T -> 0.1uF; device hermes:EMK107BBJ106MA-T_CAPC1608X95N -> rcl:C0603
- C14: value CL21B104KBCNNNC -> 10uF; device hermes:CAPC2012X140N -> rcl:C0603
- C2: value EMK107BBJ106MA-T -> 1uF; device hermes:EMK107BBJ106MA-T_CAPC1608X95N -> rcl:C0603
- C3: value GMK107AB7105KAHT -> 1uF; device hermes:CAPC1608X90N -> rcl:C0603
- C8: value CL21B104KBCNNNC -> 4.7uF; device hermes:CAPC2012X140N -> rcl:C0603
- Q2: value MMBT2222A -> BC849SMD; device hermes:SOT23 -> transistor-npn:SOT23-BEC
- Q3: value MMBT2222A -> FDN360P; device hermes:SOT23 -> transistor-power:SUPER-SOT3
- R1: value ERJ-XGNF4701Y -> 100k; device hermes:RESC1005X40 -> rcl:R0603
- R10, R17, R18, R19, R20, R21, R9: value RP73PF1J10KBTDF -> 10k; device hermes:RESC1608X50N -> rcl:R0603
- R11, R22: value RP73PF1J10KBTDF -> 4.7k; device hermes:RESC1608X50N -> rcl:R0603
- R15, R5: value ERJ-XGNF4701Y -> 4.7k; device hermes:RESC1005X40 -> rcl:R0603
- R2: value 1k -> 4.7k
- R23: value RP73PF1J10KBTDF -> 100k; device hermes:RESC1608X50N -> rcl:R0603
- R3, R7: value CPF0402B100KE1 -> 100k; device hermes:RESC1005X35N -> rcl:R0603
- R4, R8: value CPF0402B100KE1 -> 10k; device hermes:RESC1005X35N -> rcl:R0603
- moved R5 267.0 mm to (-17.1, -197.0), flipped to the top
- moved C8 253.7 mm to (-17.1, -187.1), flipped to the top
- moved R11 240.2 mm to (-17.1, -192.0)
- moved C14 231.4 mm to (-17.1, -172.2), turned to 0 degrees
- moved C5 225.2 mm to (-17.1, -182.1), flipped to the top, turned to 0 degrees
- moved C6 224.0 mm to (-17.1, -201.9)
- moved C7 219.9 mm to (-17.1, -177.2), flipped to the top, turned to 0 degrees
- moved Q3 216.6 mm to (-16.4, -165.7)
- moved R15 201.8 mm to (-17.1, -133.7)
- moved R22 179.3 mm to (-17.1, -128.8)
- moved Q2 176.8 mm to (-16.0, -122.3)
- moved R21 166.2 mm to (-17.1, -108.2)
- moved R10 157.4 mm to (-17.1, -103.3), turned to 0 degrees
- moved R9 153.6 mm to (-17.1, -98.3), turned to 0 degrees
- moved R20 137.5 mm to (-17.1, -78.5), turned to 0 degrees
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Connections:
- removed net N$11: BLUE1.2, R11.1
- removed net N$13: BLUE2.2, R12.1
- removed net N$14: BLUE3.2, R13.1
- removed net N$15: BLUE4.2, R14.1
- net 3.3V: now also C10.1, C4.1, C6.1, Q3.2, R18.2, R20.1, R22.2, R4.1, U3.7; no longer C13.1, C3.1, R16.2, R18.1, R20.2, R23.2, U7.2
- net CONFIG: now also R8.2; no longer R10.2
- net DTR: now also Q5.E, R10.1; no longer Q2.2, R22.2
- net ESP_RST: now also C3.1, Q2.C, R20.2; no longer C10.1, Q3.3, R23.1
- net GND: now also C11.2, LED2.C, LED3.C, LED4.C, LED5.C, R1.1, R2.2, R5.2, R7.1; no longer BLUE1.1, BLUE2.1, BLUE3.1, BLUE4.1, C9.2, R1.2, R10.1, R3.1, R6.2
- net GPSENABLE: now also Q3.1; no longer U7.1
- net GPSRESET: now also R11.1; no longer R5.1
- net IO0: now also Q5.C; no longer Q2.3
- net IO13: now also R23.1, R7.2; no longer R7.1, R8.2
- net LED1: now also LED2.A; no longer R11.2
- net LED2: now also LED3.A; no longer R12.2
- net LED3: now also LED4.A; no longer R13.2
- net LED4: now also LED5.A; no longer R14.2
- net N$1: now also R2.1; no longer R1.1
- net N$10: now also R17.2; no longer R18.2
- net N$16: now also C13.1; no longer C14.1
- net N$18: now also R18.1; no longer R20.1
- net N$19: now also Q2.B, R10.2; no longer Q3.1, R22.1
- net N$2: now also R24.2; no longer R2.2
- net N$20: now also Q5.B, R21.2; no longer Q2.1, R21.1
- net N$3: now also LED1.C, R24.1; no longer D1.C, R2.1
- net N$4: now also C1.1, Q4.3, R3.1; no longer C4.1, R4.1, U6.3
- net N$5: now also R3.2; no longer R4.2
- net N$6: now also C14.1, Q3.3; no longer C5.1, U7.3
- net N$7: now also C5.1; no longer C9.1
- net N$8: now also R11.2, R5.1; no longer R5.2, R6.1
- net N$9: now also R4.2; no longer R17.2
- net REGIN: no longer C6.1, U3.7
- net RTS: now also Q2.E, R21.1; no longer Q3.2, R21.2
- net SCL: now also R22.1; no longer R15.1
- net SDA: now also R15.1; no longer R16.1
- net VCC: now also LED1.A, Q4.1, R1.2; no longer D1.A, R3.2, U6.1
- net V_BATT: now also C11.1, Q4.2, R23.2; no longer C1.1, R7.2, U6.2
Routing:
- net GND: track 404.0 -> 319.5 mm, vias 40 -> 38
- net N$7: track 87.2 -> 27.7 mm
- net 3.3V: track 322.2 -> 274.2 mm, vias 15 -> 13
- net N$6: track 16.7 -> 0.79 mm
- net N$4: track 14.7 -> 1.70 mm
- net N$19: track 7.75 -> 0.00 mm, vias 2 -> 0
- net V_BATT: track 13.1 -> 5.95 mm
- net N$20: track 6.66 -> 0.00 mm, vias 2 -> 0
- net ESP_RST: track 86.3 -> 80.7 mm
- net RTS: track 87.9 -> 82.7 mm
- net DTR: track 81.0 -> 76.2 mm
- net N$10: track 4.67 -> 0.00 mm
- net VCC: track 30.9 -> 26.5 mm
- net SDA: track 163.6 -> 159.8 mm
- net USER: track 93.5 -> 90.0 mm
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