File: hermes-control.brd (EAGLE design)
At the start: 110 x 50 mm, 61 parts, among them J3 2201778-1, Q1 MMBT2222A, Q2 BC849SMD, Q3 FDN360P, Q4 FDN360P, Q5 BC849SMD, U1 LSM9DS1TR, U2 ESP32-WROOM-32D, U3 CP2104-F03-GM, U4 AP2112K-3.3TRG1, U5 MCP73831-2ACI/MC

Commit message: addresed issue comments
Parts:
- added D1: BAS40, diode:SOT23
- added Q6: MMBT2222A, hermes:SOT23
- added R12, R14, R6: 1k, rcl:R0603
- added R13: 27k, rcl:R0603
- added U$2: JST-GH-3VERT, BlueRobotics-JST-GH:JST-GH-TOP-3
Connections:
- new net N$11: U3.8
- new net N$13: Q6.1, R13.1, R6.2
- new net N$14: Q6.3, R12.1
- new net N$15: R6.1, U$2.2
- new net W_ENABLE: Q6.2, R14.2
- net 3.3V: now also R12.2, R13.2; no longer U3.8
- net GND: now also R14.1, U$2.3
- net N$4: now also D1.3
- net VCC: now also D1.1, U$2.1
Changed lines of the file:
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@@
 <attribute name="VALUE" x="-17.78" y="-203.835" size="1.27" layer="27"/>
 </element>
+<element name="D1" library="diode" library_urn="urn:adsk.eagle:library:210" package="SOT23" package3d_urn="urn:adsk.eagle:package:43389/2" value="BAS40" x="-16.002" y="-208.407" smashed="yes">
+<attribute name="NAME" x="-17.907" y="-206.502" size="1.27" layer="25"/>
+<attribute name="VALUE" x="-17.907" y="-211.582" size="1.27" layer="27"/>
+</element>
+<element name="R6" library="rcl" library_urn="urn:adsk.eagle:library:334" package="R0603" package3d_urn="urn:adsk.eagle:package:23555/3" value="1k" x="-12.192" y="-228.219" smashed="yes">
+<attribute name="NAME" x="-12.827" y="-227.584" size="1.27" layer="25"/>
+<attribute name="SPICEPREFIX" value="R" x="-17.145" y="-214.884" size="1.778" layer="27" display="off"/>
+<attribute name="VALUE" x="-12.827" y="-230.124" size="1.27" layer="27"/>
+</element>
+<element name="Q6" library="hermes" package="SOT23" value="MMBT2222A" x="-15.24" y="-216.027" smashed="yes">
+<attribute name="DIGIKEY" value="568-4509-6-ND" x="-15.24" y="-221.361" size="1.778" layer="27" display="off"/>
+<attribute name="ELEMENT14" value="1757934" x="-15.24" y="-221.361" size="1.778" layer="27" display="off"/>
+<attribute name="NAME" x="-16.12959375" y="-213.993640625" size="1.27085" layer="25"/>
+<attribute name="VALUE" x="-18.16255" y="-220.02961875" size="1.27066875" layer="27"/>
+</element>
+<element name="R12" library="rcl" library_urn="urn:adsk.eagle:library:334" package="R0603" package3d_urn="urn:adsk.eagle:package:23555/3" value="1k" x="-17.145" y="-223.266" smashed="yes">
+<attribute name="NAME" x="-17.78" y="-222.631" size="1.27" layer="25"/>
+<attribute name="SPICEPREFIX" value="R" x="-17.145" y="-228.6" size="1.778" layer="27" display="off"/>
+<attribute name="VALUE" x="-17.78" y="-225.171" size="1.27" layer="27"/>
+</element>
+<element name="R13" library="rcl" library_urn="urn:adsk.eagle:library:334" package="R0603" package3d_urn="urn:adsk.eagle:package:23555/3" value="27k" x="-12.192" y="-223.266" smashed="yes">
+<attribute name="NAME" x="-12.827" y="-222.631" size="1.27" layer="25"/>
+<attribute name="SPICEPREFIX" value="R" x="-17.145" y="-233.553" size="1.778" layer="27" display="off"/>
+<attribute name="VALUE" x="-12.827" y="-225.171" size="1.27" layer="27"/>
+</element>
+<element name="R14" library="rcl" library_urn="urn:adsk.eagle:library:334" package="R0603" package3d_urn="urn:adsk.eagle:package:23555/3" value="1k" x="-17.145" y="-228.219" smashed="yes">
+<attribute name="NAME" x="-17.78" y="-227.584" size="1.27" layer="25"/>
+<attribute name="SPICEPREFIX" value="R" x="-17.145" y="-238.506" size="1.778" layer="27" display="off"/>
+<attribute name="VALUE" x="-17.78" y="-230.124" size="1.27" layer="27"/>
+</element>
+<element name="U$2" library="BlueRobotics-JST-GH" package="JST-GH-TOP-3" value="JST-GH-3VERT" x="-16.002" y="-231.648" smashed="yes"/>
 </elements>
 <signals>
@@
 <contactref element="C13" pad="2"/>
 <contactref element="R7" pad="1"/>
-<contactref element="R9" pad="1"/>
-<contactref element="R8" pad="1"/>
 <contactref element="LED2" pad="C"/>
 <contactref element="LED3" pad="C"/>
@@
 <contactref element="R5" pad="2"/>
 <contactref element="C6" pad="2"/>
+<contactref element="R9" pad="1"/>
+<contactref element="R8" pad="1"/>
+<contactref element="R14" pad="1"/>
+<contactref element="U$2" pad="3"/>
+<wire x1="-17.995" y1="-228.219" x2="-16.002" y2="-231.648" width="0" layer="19" extent="1-1"/>
+<wire x1="-16.295" y1="-201.93" x2="-17.995" y2="-228.219" width="0" layer="19" extent="1-1"/>
 <wire x1="-16.295" y1="-196.977" x2="-16.295" y2="-201.93" width="0" layer="19" extent="1-1"/>
 <wire x1="-16.295" y1="-187.071" x2="-16.295" y2="-196.977" width="0" layer="19" extent="1-1"/>
@@
 <contactref element="U1" pad="23"/>
 <wire x1="24.045" y1="28.89" x2="24.6" y2="29.445" width="0.1524" layer="1"/>
-<contactref element="U3" pad="8"/>
 <wire x1="38.165" y1="28.88" x2="38.165" y2="29.2032875" width="0.1524" layer="1"/>
 <wire x1="38.165" y1="29.2032875" x2="35.0982875" y2="32.27" width="0.1524" layer="1"/>
@@
 <wire x1="19.85064375" y1="20.2664" x2="19.7114" y2="20.40564375" width="0.1524" layer="1"/>
 <wire x1="19.7114" y1="20.40564375" x2="19.7114" y2="20.7636" width="0.1524" layer="1"/>
-<wire x1="19.7114" y1="20.7636" x2="19.57" y2="20.905" width="0.1524" layer="1"/>
 <wire x1="21.78935625" y1="20.2664" x2="19.85064375" y2="20.2664" width="0.1524" layer="1"/>
 <wire x1="25.4" y1="35.5092" x2="25.4" y2="27.94" width="0.1524" layer="16"/>
@@
 <contactref element="C6" pad="1"/>
 <wire x1="19.07" y1="20.905" x2="18.72" y2="20.555" width="0.1524" layer="1"/>
+<contactref element="R12" pad="2"/>
+<contactref element="R13" pad="2"/>
+<wire x1="-11.342" y1="-223.266" x2="-16.295" y2="-223.266" width="0" layer="19" extent="1-1"/>
+<wire x1="-17.995" y1="-201.93" x2="-16.295" y2="-223.266" width="0" layer="19" extent="1-1"/>
 <wire x1="-15.433" y1="-166.835" x2="-17.995" y2="-201.93" width="0" layer="19" extent="1-1"/>
 <wire x1="-16.295" y1="-133.731" x2="-15.433" y2="-166.835" width="0" layer="19" extent="1-1"/>
@@
 <wire x1="-17.995" y1="-28.956" x2="-17.995" y2="-33.909" width="0" layer="19" extent="1-1"/>
 <wire x1="18.72" y1="20.555" x2="-17.995" y2="-28.956" width="0" layer="19" extent="1-1"/>
-<wire x1="19.57" y1="20.905" x2="19.07" y2="20.905" width="0" layer="19" extent="1-1"/>
+<wire x1="19.7114" y1="20.7636" x2="19.07" y2="20.905" width="0" layer="19" extent="1-1"/>
 <wire x1="22.9489375" y1="39.8136" x2="22.987" y2="37.9222" width="0" layer="19" extent="1-16"/>
 <wire x1="28.46" y1="32.27" x2="25.4" y2="35.5092" width="0" layer="19" extent="1-16"/>
@@
 <contactref element="R1" pad="2"/>
 <contactref element="Q4" pad="1"/>
-<wire x1="11.3595875" y1="34.29" x2="15.113" y2="33.0962" width="0" layer="19" extent="1-1"/>
-<wire x1="-15.621" y1="-2.574" x2="11.4" y2="20.505" width="0" layer="19" extent="1-1"/>
-<wire x1="-16.295" y1="-6.096" x2="-15.621" y2="-2.574" width="0" layer="19" extent="1-1"/>
-<wire x1="-17.333" y1="-13.673" x2="-16.295" y2="-6.096" width="0" layer="19" extent="1-1"/>
+<contactref element="D1" pad="1"/>
+<contactref element="U$2" pad="1"/>
+<wire x1="-16.952" y1="-209.507" x2="-13.502" y2="-231.648" width="0" layer="19" extent="1-1"/>
+<wire x1="-17.333" y1="-13.673" x2="-16.952" y2="-209.507" width="0" layer="19" extent="1-1"/>
+<wire x1="-16.295" y1="-6.096" x2="-17.333" y2="-13.673" width="0" layer="19" extent="1-1"/>
+<wire x1="-15.621" y1="-2.574" x2="-16.295" y2="-6.096" width="0" layer="19" extent="1-1"/>
+<wire x1="11.4" y1="20.505" x2="-15.621" y2="-2.574" width="0" layer="19" extent="1-1"/>
+<wire x1="15.113" y1="33.0962" x2="11.3595875" y2="34.29" width="0" layer="19" extent="1-1"/>
 </signal>
 <signal name="N$2">
@@
 <contactref element="C1" pad="1"/>
 <contactref element="R3" pad="1"/>
-<wire x1="-16.383" y1="-11.473" x2="19.979" y2="28.89" width="0" layer="19" extent="1-1"/>
-<wire x1="-17.995" y1="-19.05" x2="-16.383" y2="-11.473" width="0" layer="19" extent="1-1"/>
-<wire x1="-17.995" y1="-24.003" x2="-17.995" y2="-19.05" width="0" layer="19" extent="1-1"/>
+<contactref element="D1" pad="3"/>
+<wire x1="-17.995" y1="-24.003" x2="-16.002" y2="-207.307" width="0" layer="19" extent="1-1"/>
+<wire x1="-17.995" y1="-19.05" x2="-17.995" y2="-24.003" width="0" layer="19" extent="1-1"/>
+<wire x1="-16.383" y1="-11.473" x2="-17.995" y2="-19.05" width="0" layer="19" extent="1-1"/>
+<wire x1="19.979" y1="28.89" x2="-16.383" y2="-11.473" width="0" layer="19" extent="1-1"/>
 </signal>
 <signal name="N$5">
@@
 <wire x1="52.959" y1="21.336" x2="52.233" y2="22.062" width="0.1524" layer="1"/>
 <wire x1="52.233" y1="22.062" x2="50.471" y2="22.062" width="0.1524" layer="1"/>
-<contactref element="C3" pad="1"/>
 <contactref element="R20" pad="2"/>
 <contactref element="Q2" pad="C"/>
+<contactref element="C3" pad="1"/>
 <wire x1="-16.295" y1="-78.486" x2="-16.002" y2="-121.201" width="0" layer="19" extent="1-1"/>
 <wire x1="-17.995" y1="-38.862" x2="-16.295" y2="-78.486" width="0" layer="19" extent="1-1"/>
@@
 <wire x1="56.52" y1="57.785" x2="-16.295" y2="-192.024" width="0" layer="19" extent="1-16"/>
 </signal>
+<signal name="N$11">
+<contactref element="U3" pad="8"/>
+</signal>
+<signal name="N$13">
+<contactref element="R6" pad="2"/>
+<contactref element="Q6" pad="1"/>
+<contactref element="R13" pad="1"/>
+<wire x1="-13.042" y1="-223.266" x2="-11.342" y2="-228.219" width="0" layer="19" extent="1-1"/>
+<wire x1="-16.19" y1="-217.127" x2="-13.042" y2="-223.266" width="0" layer="19" extent="1-1"/>
+</signal>
+<signal name="N$14">
+<contactref element="R12" pad="1"/>
+<contactref element="Q6" pad="3"/>
+<wire x1="-15.24" y1="-214.927" x2="-17.995" y2="-223.266" width="0" layer="19" extent="1-1"/>
+</signal>
+<signal name="W_ENABLE">
+<contactref element="R14" pad="2"/>
+<contactref element="Q6" pad="2"/>
+<wire x1="-14.29" y1="-217.127" x2="-16.295" y2="-228.219" width="0" layer="19" extent="1-1"/>
+</signal>
+<signal name="N$15">
+<contactref element="U$2" pad="2"/>
+<contactref element="R6" pad="1"/>
+<wire x1="-13.042" y1="-228.219" x2="-14.752" y2="-231.648" width="0" layer="19" extent="1-1"/>
+</signal>
 </signals>
