File: hermes-control.sch (EAGLE design)
At the start: 65 parts, among them J3 2201778-1, Q1 MMBT2222A, Q2 MMBT2222A, Q3 MMBT2222A, U1 LSM9DS1TR, U2 ESP32-WROOM-32D, U3 CP2104-F03-GM, U4 AP2112K-3.3TRG1, U5 MCP73831-2ACI/MC, U6 DMG3415U-7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

Commit message: lets clean this up
Parts:
- added R24: 1k, rcl:R-US_R0603
- R2: value CPF0402B1K0E1 -> 1k; device hermes:CPF0402B1K0E1 -> rcl:R-US_R0603
Changed lines of the file:
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@@
 <grid distance="0.1" unitdist="inch" unit="inch" style="lines" multiple="1" display="no" altdistance="0.01" altunitdist="inch" altunit="inch"/>
 <layers>
-<layer number="1" name="Top" color="4" fill="1" visible="no" active="no"/>
-<layer number="16" name="Bottom" color="1" fill="1" visible="no" active="no"/>
-<layer number="17" name="Pads" color="2" fill="1" visible="no" active="no"/>
-<layer number="18" name="Vias" color="2" fill="1" visible="no" active="no"/>
-<layer number="19" name="Unrouted" color="6" fill="1" visible="no" active="no"/>
-<layer number="20" name="Dimension" color="24" fill="1" visible="no" active="no"/>
-<layer number="21" name="tPlace" color="7" fill="1" visible="no" active="no"/>
-<layer number="22" name="bPlace" color="7" fill="1" visible="no" active="no"/>
-<layer number="23" name="tOrigins" color="15" fill="1" visible="no" active="no"/>
-<layer number="24" name="bOrigins" color="15" fill="1" visible="no" active="no"/>
-<layer number="25" name="tNames" color="7" fill="1" visible="no" active="no"/>
-<layer number="26" name="bNames" color="7" fill="1" visible="no" active="no"/>
-<layer number="27" name="tValues" color="7" fill="1" visible="no" active="no"/>
-<layer number="28" name="bValues" color="7" fill="1" visible="no" active="no"/>
+<layer number="1" name="Top" color="4" fill="1" visible="yes" active="no"/>
+<layer number="16" name="Bottom" color="1" fill="1" visible="yes" active="no"/>
+<layer number="17" name="Pads" color="2" fill="1" visible="yes" active="no"/>
+<layer number="18" name="Vias" color="2" fill="1" visible="yes" active="no"/>
+<layer number="19" name="Unrouted" color="6" fill="1" visible="yes" active="no"/>
+<layer number="20" name="Dimension" color="24" fill="1" visible="yes" active="no"/>
+<layer number="21" name="tPlace" color="7" fill="1" visible="yes" active="no"/>
+<layer number="22" name="bPlace" color="7" fill="1" visible="yes" active="no"/>
+<layer number="23" name="tOrigins" color="15" fill="1" visible="yes" active="no"/>
+<layer number="24" name="bOrigins" color="15" fill="1" visible="yes" active="no"/>
+<layer number="25" name="tNames" color="7" fill="1" visible="yes" active="no"/>
+<layer number="26" name="bNames" color="7" fill="1" visible="yes" active="no"/>
+<layer number="27" name="tValues" color="7" fill="1" visible="yes" active="no"/>
+<layer number="28" name="bValues" color="7" fill="1" visible="yes" active="no"/>
 <layer number="29" name="tStop" color="7" fill="3" visible="no" active="no"/>
 <layer number="30" name="bStop" color="7" fill="6" visible="no" active="no"/>
@@
 <layer number="35" name="tGlue" color="7" fill="4" visible="no" active="no"/>
 <layer number="36" name="bGlue" color="7" fill="5" visible="no" active="no"/>
-<layer number="37" name="tTest" color="7" fill="1" visible="no" active="no"/>
-<layer number="38" name="bTest" color="7" fill="1" visible="no" active="no"/>
+<layer number="37" name="tTest" color="7" fill="1" visible="yes" active="no"/>
+<layer number="38" name="bTest" color="7" fill="1" visible="yes" active="no"/>
 <layer number="39" name="tKeepout" color="4" fill="11" visible="no" active="no"/>
 <layer number="40" name="bKeepout" color="1" fill="11" visible="no" active="no"/>
@@
 <layer number="44" name="Drills" color="7" fill="1" visible="no" active="no"/>
 <layer number="45" name="Holes" color="7" fill="1" visible="no" active="no"/>
-<layer number="46" name="Milling" color="3" fill="1" visible="no" active="no"/>
-<layer number="47" name="Measures" color="7" fill="1" visible="no" active="no"/>
-<layer number="48" name="Document" color="7" fill="1" visible="no" active="no"/>
-<layer number="49" name="Reference" color="7" fill="1" visible="no" active="no"/>
-<layer number="50" name="dxf" color="7" fill="1" visible="no" active="no"/>
-<layer number="51" name="tDocu" color="7" fill="1" visible="no" active="no"/>
-<layer number="52" name="bDocu" color="7" fill="1" visible="no" active="no"/>
-<layer number="53" name="tGND_GNDA" color="7" fill="9" visible="no" active="no"/>
-<layer number="54" name="bGND_GNDA" color="1" fill="9" visible="no" active="no"/>
-<layer number="56" name="wert" color="7" fill="1" visible="no" active="no"/>
-<layer number="57" name="tCAD" color="7" fill="1" visible="no" active="no"/>
-<layer number="59" name="tCarbon" color="7" fill="1" visible="no" active="no"/>
-<layer number="60" name="bCarbon" color="7" fill="1" visible="no" active="no"/>
+<layer number="46" name="Milling" color="3" fill="1" visible="yes" active="no"/>
+<layer number="47" name="Measures" color="7" fill="1" visible="yes" active="no"/>
+<layer number="48" name="Document" color="7" fill="1" visible="yes" active="no"/>
+<layer number="49" name="Reference" color="7" fill="1" visible="yes" active="no"/>
+<layer number="50" name="dxf" color="7" fill="1" visible="yes" active="no"/>
+<layer number="51" name="tDocu" color="7" fill="1" visible="yes" active="no"/>
+<layer number="52" name="bDocu" color="7" fill="1" visible="yes" active="no"/>
+<layer number="53" name="tGND_GNDA" color="7" fill="9" visible="yes" active="no"/>
+<layer number="54" name="bGND_GNDA" color="1" fill="9" visible="yes" active="no"/>
+<layer number="56" name="wert" color="7" fill="1" visible="yes" active="no"/>
+<layer number="57" name="tCAD" color="7" fill="1" visible="yes" active="no"/>
+<layer number="59" name="tCarbon" color="7" fill="1" visible="yes" active="no"/>
+<layer number="60" name="bCarbon" color="7" fill="1" visible="yes" active="no"/>
 <layer number="88" name="SimResults" color="9" fill="1" visible="yes" active="yes"/>
 <layer number="89" name="SimProbes" color="9" fill="1" visible="yes" active="yes"/>
@@
 <part name="SUPPLY2" library="SparkFun-PowerSymbols" library_urn="urn:adsk.eagle:library:530" deviceset="VCC" device=""/>
 <part name="D1" library="hermes" deviceset="598-8040-107F" device="" value="Yellow"/>
-<part name="R2" library="hermes" deviceset="CPF0402B1K0E1" device="" value="CPF0402B1K0E1"/>
+<part name="R2" library="rcl" library_urn="urn:adsk.eagle:library:334" deviceset="R-US_" device="R0603" package3d_urn="urn:adsk.eagle:package:23555/3" value="1k"/>
 <part name="SUPPLY3" library="SparkFun-PowerSymbols" library_urn="urn:adsk.eagle:library:530" deviceset="3.3V" device=""/>
 <part name="C2" library="hermes" deviceset="EMK107BBJ106MA-T" device="" value="EMK107BBJ106MA-T"/>
@@
 <part name="SUPPLY25" library="SparkFun-PowerSymbols" library_urn="urn:adsk.eagle:library:530" deviceset="3.3V" device=""/>
 <part name="R23" library="hermes" deviceset="RP73PF1J10KBTDF" device="" value="RP73PF1J10KBTDF"/>
+<part name="R24" library="rcl" library_urn="urn:adsk.eagle:library:334" deviceset="R-US_" device="R0603" package3d_urn="urn:adsk.eagle:package:23555/3" value="1k"/>
 </parts>
 <sheets>
@@
 <instance part="R23" gate="G$1" x="375.92" y="76.2" smashed="yes" rot="R180">
 <attribute name="NAME" x="375.92" y="74.676" size="1.778" layer="95" font="vector" rot="R180" align="bottom-center"/>
+</instance>
+<instance part="R24" gate="G$1" x="93.98" y="144.78" smashed="yes">
+<attribute name="NAME" x="90.17" y="146.2786" size="1.778" layer="95"/>
+<attribute name="VALUE" x="90.17" y="141.478" size="1.778" layer="96"/>
 </instance>
 </instances>
@@
 packages will not be understood (or retained) with this version.
 </note>
+<note version="8.4" severity="warning">
+Since Version 8.4, EAGLE supports properties for SPICE simulation.
+Probes in schematics and SPICE mapping objects found in parts and library devices
+will not be understood with this version. Update EAGLE to the latest version
+for full support of SPICE simulation.
+</note>
 </compatibility>

Commit message: replaced all componets with generics
Parts:
- removed BLUE1, BLUE2, BLUE3, BLUE4: LTST-C190TBKT, hermes:LTST-C190TBKT
- removed C9: JMK107BJ475KA-T, hermes:JMK107BJ475KA-T
- removed D1: Yellow, hermes:598-8040-107F
- removed R12, R13, R14: RP73PF1J10KBTDF, hermes:RP73PF1J10KBTDF
- removed R16, R6: ERJ-XGNF4701Y, hermes:ERJ-XGNF4701Y
- removed U6, U7: DMG3415U-7, SnapEDA-Library:DMG3415U-7
- added C11: 10uF, rcl:C-USC0603
- added LED1: Yellow, led:LEDCHIPLED_0805
- added LED2, LED3, LED5: Blue, led:LEDCHIPLED_0805
- added LED4: BLue, led:LEDCHIPLED_0805
- added Q4: FDN360P, transistor-power:FDN360P
- added Q5: BC849SMD, transistor-npn:BC849SMD
- C1, C4, C6: value EMK107BBJ106MA-T -> 10uF; device hermes:EMK107BBJ106MA-T -> rcl:C-USC0603
- C10: value GMK107AB7105KAHT -> 10uF; device hermes:GMK107AB7105KAHT -> rcl:C-USC0603
- C12, C5: value CL21B104KBCNNNC -> 0.1uF; device hermes:CL21B104KBCNNNC -> rcl:C-USC0603
- C13, C7: value EMK107BBJ106MA-T -> 0.1uF; device hermes:EMK107BBJ106MA-T -> rcl:C-USC0603
- C14: value CL21B104KBCNNNC -> 10uF; device hermes:CL21B104KBCNNNC -> rcl:C-USC0603
- C2: value EMK107BBJ106MA-T -> 1uF; device hermes:EMK107BBJ106MA-T -> rcl:C-USC0603
- C3: value GMK107AB7105KAHT -> 1uF; device hermes:GMK107AB7105KAHT -> rcl:C-USC0603
- C8: value CL21B104KBCNNNC -> 4.7uF; device hermes:CL21B104KBCNNNC -> rcl:C-USC0603
- Q2: value MMBT2222A -> BC849SMD; device hermes:MMBT2222A -> transistor-npn:BC849SMD
- Q3: value MMBT2222A -> FDN360P; device hermes:MMBT2222A -> transistor-power:FDN360P
- R1: value ERJ-XGNF4701Y -> 100k; device hermes:ERJ-XGNF4701Y -> rcl:R-US_R0603
- R10, R17, R18, R19, R20, R21, R9: value RP73PF1J10KBTDF -> 10k; device hermes:RP73PF1J10KBTDF -> rcl:R-US_R0603
- R11, R22: value RP73PF1J10KBTDF -> 4.7k; device hermes:RP73PF1J10KBTDF -> rcl:R-US_R0603
- R15, R5: value ERJ-XGNF4701Y -> 4.7k; device hermes:ERJ-XGNF4701Y -> rcl:R-US_R0603
- R2: value 1k -> 4.7k
- R23: value RP73PF1J10KBTDF -> 100k; device hermes:RP73PF1J10KBTDF -> rcl:R-US_R0603
- R3, R7: value CPF0402B100KE1 -> 100k; device hermes:CPF0402B100KE1 -> rcl:R-US_R0603
- R4, R8: value CPF0402B100KE1 -> 10k; device hermes:CPF0402B100KE1 -> rcl:R-US_R0603
Connections:
- removed net N$11: BLUE1.A2, R11.1
- removed net N$13: BLUE2.A2, R12.1
- removed net N$14: BLUE3.A2, R13.1
- removed net N$15: BLUE4.A2, R14.1
- net 3.3V: now also C10.1, C4.1, C6.1, Q3.S, R18.2, R20.1, R22.2, R4.1, U3.REGIN; no longer C13.1, C3.1, R16.2, R18.1, R20.2, R23.2, U7.S
- net CONFIG: now also R8.2; no longer R10.2
- net DTR: now also Q5.E, R10.1; no longer Q2.E, R22.2
- net ESP_RST: now also C3.1, Q2.C, R20.2; no longer C10.1, Q3.C, R23.1
- net GND: now also C11.2, LED2.C, LED3.C, LED4.C, LED5.C, R1.1, R2.2, R5.2, R7.1; no longer BLUE1.K2, BLUE2.K2, BLUE3.K2, BLUE4.K2, C9.2, R1.2, R10.1, R3.1, R6.2
- net GPSENABLE: now also Q3.G; no longer U7.G
- net GPSRESET: now also R11.1; no longer R5.1
- net IO0: now also Q5.C; no longer Q2.C
- net IO13: now also R23.1, R7.2; no longer R7.1, R8.2
- net LED1: now also LED2.A; no longer R11.2
- net LED2: now also LED3.A; no longer R12.2
- net LED3: now also LED4.A; no longer R13.2
- net LED4: now also LED5.A; no longer R14.2
- net N$1: now also R2.1; no longer R1.1
- net N$10: now also R17.2; no longer R18.2
- net N$16: now also C13.1; no longer C14.1
- net N$18: now also R18.1; no longer R20.1
- net N$19: now also Q2.B, R10.2; no longer Q3.B, R22.1
- net N$2: now also R24.2; no longer R2.2
- net N$20: now also Q5.B, R21.2; no longer Q2.B, R21.1
- net N$3: now also LED1.C, R24.1; no longer D1.C, R2.1
- net N$4: now also C1.1, Q4.D, R3.1; no longer C4.1, R4.1, U6.D
- net N$5: now also R3.2; no longer R4.2
- net N$6: now also C14.1, Q3.D; no longer C5.1, U7.D
- net N$7: now also C5.1; no longer C9.1
- net N$8: now also R11.2, R5.1; no longer R5.2, R6.1
- net N$9: now also R4.2; no longer R17.2
- net REGIN: no longer C6.1, U3.REGIN
- net RTS: now also Q2.E, R21.1; no longer Q3.E, R21.2
- net SCL: now also R22.1; no longer R15.1
- net SDA: now also R15.1; no longer R16.1
- net VCC: now also LED1.A, Q4.G, R1.2; no longer D1.A, R3.2, U6.G
- net V_BATT: now also C11.1, Q4.S, R23.2; no longer C1.1, R7.2, U6.S
Other:
- moved on the sheet: C1, C10, C12, C13, C14, C2, C3, C4, C5, C6, C7, C8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

Commit message: addresed issue comments
Parts:
- added D1: BAS40, diode:BAS40
- added Q6: MMBT2222A, hermes:MMBT2222A
- added R12, R14, R6: 1k, rcl:R-US_R0603
- added R13: 27k, rcl:R-US_R0603
- added U$2: JST-GH-3VERT, BlueRobotics-JST-GH:JST-GH-3VERT
Connections:
- new net N$11: U3.VBUS
- new net N$13: Q6.B, R13.1, R6.2
- new net N$14: Q6.C, R12.1
- new net N$15: R6.1, U$2.2
- new net W_ENABLE: Q6.E, R14.2
- net 3.3V: now also R12.2, R13.2; no longer U3.VBUS
- net GND: now also R14.1, U$2.3
- net N$4: now also D1.C
- net VCC: now also D1.A, U$2.1
Other:
- moved on the sheet: C3, J3, LED2, LED3, LED4, LED5, R15, R20, R8, R9, S1, S2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

Commit message: updated resistors and addressed comments
Parts:
- removed R19: 10k, rcl:R-US_R0603
- added C15: 100uF, rcl:C-USC0603
- added C9: 10uF, rcl:C-USC0603
- added Q7: FDN360P, transistor-power:FDN360P
- added R16: 1k, rcl:R-US_R0603
- R14: value 1k -> 10k
- R17, R18, R4: value 10k -> 1k
- R23: value 100k -> 33k
Connections:
- removed net REGIN: U3.VDD, U3.VIO
- new net N$21: LED4.A, R17.1
- new net N$22: LED5.A, R18.1
- new net N$23: Q7.G
- new net VCCIO: C2.1, C4.1, Q7.D, R20.1, U2.3V3, U4.VOUT
- net 3.3V: now also Q3.D, Q7.S, U1.CS_A/G, U1.CS_M, U1.SDO_A/G, U1.SDO_M, U3.VDD, U3.VIO; no longer C2.1, C4.1, Q3.S, R17.1, R18.2, R19.2, R20.1, R4.1, U2.3V3, U4.VOUT
- net GND: now also C15.2, C9.2
- net LED1: now also R4.2; no longer LED2.A
- net LED2: now also R16.2; no longer LED3.A
- net LED3: now also R17.2; no longer LED4.A
- net LED4: now also R18.2; no longer LED5.A
- net N$10: now also C15.1, U1.C1; no longer R17.2, U1.CS_M
- net N$17: now also LED2.A, R4.1; no longer R19.1, U1.SDO_A/G
- net N$18: now also LED3.A, R16.1; no longer R18.1, U1.SDO_M
- net N$4: now also Q4.S; no longer Q4.D
- net N$6: now also Q3.S; no longer Q3.D
- net N$9: now also C9.1, U1.CAP; no longer R4.2, U1.CS_A/G
- net V_BATT: now also Q4.D; no longer Q4.S
Other:
- moved on the sheet: LED2, LED3, LED4, LED5, R17, R18, R4

Commit message: updated GPIO
Connections:
- net IO0 renamed PGM
- net USBRX renamed RX0
- net USBTX renamed TX0
- removed net DIN: J3.CMD, U2.SDI/SD1
- removed net DOUT: J3.DAT0, U2.SDO/SD0
- removed net GPSENABLE: Q3.G, U2.IO23
- removed net GPSRX: U$1.RXD1, U2.IO19
- removed net GPSTX: U$1.TXD1, U2.IO18
- removed net N$23: Q7.G
- removed net SCLK: J3.CLK, U2.SCL/CLK
- removed net W_ENABLE: Q6.E, R14.2
- new net CLK: J3.CLK, U2.IO18
- new net GPS_EN: Q3.G, U2.IO27
- new net MISO: J3.DAT0, U2.IO19
- new net MOSI: J3.CMD, U2.IO23
- new net RL_33: Q7.G, U2.IO32
- new net RX3: U$8.3, U2.IO26
- new net TX3: U$8.2, U2.IO25
- new net WATER: Q6.E, R14.2, U2.SENSOR_VP
- net CONFIG: now also U2.SENSOR_VN; no longer U2.IO15
- net CS: now also U2.IO5; no longer U2.SCS/CMD
- net IO13: now also U2.IO34; no longer U2.IO14
- net LED1: now also U2.IO12; no longer U2.IO4
- net LED2: now also U2.IO13; no longer U2.IO5
- net LED3: now also U2.IO14; no longer U2.IO12
- net LED4: now also U2.IO15; no longer U2.IO13
- net RX1: now also U$1.TXD1, U2.IO16; no longer U$7.3, U2.SHD/SD2
- net RX2: now also U$7.3, U2.IO4; no longer U$8.3, U2.IO16
- net TX1: now also U$1.RXD1, U2.IO17; no longer U$7.2, U2.SWP/SD3
- net TX2: now also U$7.2, U2.IO2; no longer U$8.2, U2.IO17
- net USER: now also U2.IO35; no longer U2.IO2
Other:
- moved on the sheet: R23, R7, R8, R9, S1, S2
